File: Porshe_PCB.kicad_sch (KiCad schematic)
At the start: 55 parts, among them IC1 RASPBERRY_PI_PICO_W, IC2 BH1750FVI-TR, J1 TF-115, J10 Conn_01x01_Pin, J11 Conn_01x01_Pin, J12 Conn_01x01_Pin, J13 Barrel_Jack, J14 Conn_02x20_Odd_Even, J15 Conn_01x03_Pin, J16 Conn_02x20_Odd_Even, J17 Conn_01x03_Pin, J18 Conn_01x01_Pin, J19 Conn_01x01_Pin, J2 SM04B-SRSS-TB_LF__SN_, J3 Conn_02x02_Odd_Even, J4 S2B-PH-SM4-TB_LF__SN_, J5 Conn_01x01_Pin, J6 Conn_01x01_Pin, J7 Conn_01x01_Pin, J8 Conn_01x01_Pin, J9 Conn_02x04_Odd_Even, M1 Fan, Q1 DMG2305UX-7, Q2 2N3904, U1 DS3231SN

Commit message: 첫번째 완성
Parts:
- added R11, R12: 220, Resistor_SMD:R_0603_1608Metric_Pad0.98x0.95mm_HandSolder, symbol Device:R
- M1: now left out of the parts list
Connections:
- net SPI0_SCK is gone; now on net SPI1_SCK: J1.5 (CLX)
- net 3V3: no longer J15.1 (Pin_1), J17.1 (Pin_1), LED1.1 (VDD)
- net DIN_1: now also R11.1; no longer J15.2 (Pin_2)
- net DIN_2: now also R12.1; no longer J17.2 (Pin_2)
- net GND: now also J15.1 (Pin_1), J17.1 (Pin_1)
- net VSYS: now also C3.1, C4.1, J15.3 (Pin_3), J17.3 (Pin_3), LED1.1 (VDD)
- net SPI0_MISO renamed SPI1_MISO
- net SPI0_MOSI renamed SPI1_MOSI
- net SPI_SC renamed SPI1_SC
- new net: J15.2 (Pin_2), R11.2
- new net: J17.2 (Pin_2), R12.2
Other:
- note added: "Fan"
- moved on the sheet: C3, C4, J15, J18

Commit message: 오토라우딩하기전
Parts:
- removed H1: MountingHole_Pad, MountingHole:MountingHole_2.7mm_M2.5_ISO7380_Pad_TopOnly, symbol Mechanical:MountingHole_Pad
- removed J3: Conn_02x02_Odd_Even, Connector_PinSocket_2.54mm:PinSocket_2x02_P2.54mm_Vertical_SMD, symbol Connector_Generic:Conn_02x02_Odd_Even
- added H5, H6: MountingHole_Pad, MountingHole:MountingHole_2.7mm_M2.5_ISO7380_Pad_TopOnly, symbol Mechanical:MountingHole_Pad
Connections:
- net Buzz: now also J14.23 (Pin_23), J14.24 (Pin_24); no longer J16.19 (Pin_19), J16.20 (Pin_20)
- net DI: now also J14.19 (Pin_19), J14.20 (Pin_20)
- net DIN_1: now also J16.37 (Pin_37), J16.38 (Pin_38); no longer J14.31 (Pin_31), J14.32 (Pin_32)
- net DIN_2: now also J16.39 (Pin_39), J16.40 (Pin_40); no longer J14.27 (Pin_27), J14.28 (Pin_28)
- net FAN: now also J16.33 (Pin_33), J16.34 (Pin_34); no longer J14.33 (Pin_33), J14.34 (Pin_34)
- net GND: now also H5.1, H6.1
- net LED: now also J14.27 (Pin_27), J14.28 (Pin_28); no longer J16.33 (Pin_33), J16.34 (Pin_34)
- net RTC_RST: now also J16.19 (Pin_19), J16.20 (Pin_20); no longer J14.23 (Pin_23), J14.24 (Pin_24)
- net SW1: now also J14.29 (Pin_29), J14.30 (Pin_30); no longer J16.37 (Pin_37), J16.38 (Pin_38)
- net SPI0_SC: now reaches J14.37 (Pin_37), J14.38 (Pin_38)
- net SPI0_SC: now also J1.1 (DAT2), R2.1
- net SPI0_MISO: now reaches J14.39 (Pin_39), J14.40 (Pin_40)
- net SPI0_MISO: now also J1.7 (DAT0)
- net SPI1_MISO: no longer names the net of J16.21 (Pin_21), J16.22 (Pin_22)
- net SPI1_MISO: no longer J1.7 (DAT0)
- net SPI1_MOSI: no longer names the net of J16.29 (Pin_29), J16.30 (Pin_30)
- net SPI1_MOSI: no longer J1.3 (CMD)
- net SPI1_SC: no longer names the net of J16.23 (Pin_23), J16.24 (Pin_24)
- net SPI1_SC: no longer J1.1 (DAT2), R2.1
- net SPI1_SCK: no longer names the net of J16.27 (Pin_27), J16.28 (Pin_28)
- net SPI1_SCK: no longer J1.5 (CLX)
- new net SPI0_MOSI: J1.3 (CMD), J14.31 (Pin_31), J14.32 (Pin_32)
- new net SPI0_SCK: J1.5 (CLX), J14.33 (Pin_33), J14.34 (Pin_34)
Other:
- note removed: "UART"

Commit message: 주문을 위한 버전
Parts:
- C3, C4, J13, J15, J17, JP3, Q2: now left out of the parts list
Connections:
- net DI: no longer J16.17 (Pin_17), J16.18 (Pin_18)
- new net: J16.17 (Pin_17), J16.18 (Pin_18)
- no-connect marks 47 -> 49
Changed lines of the file:
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@@
   (junction (at 154.94 170.18) (diameter 0) (color 0 0 0 0)
   )
-  (junction (at 46.99 45.72) (diameter 0) (color 0 0 0 0)
-  )
   (junction (at 180.34 130.175) (diameter 0) (color 0 0 0 0)
   )
@@
   (no_connect (at 163.83 45.085))
   (no_connect (at 202.565 96.52))
+  (no_connect (at 222.885 -7.62))
   (no_connect (at 64.77 50.165))
   (no_connect (at 64.77 52.705))
@@
   (no_connect (at 163.83 65.405))
   (no_connect (at 64.77 70.485))
+  (no_connect (at 283.21 12.7))
   (no_connect (at 64.77 65.405))
   (no_connect (at 163.83 42.545))
@@
     (stroke (width 0) (type default))
   )
-  (wire (pts (xy 46.99 45.72) (xy 22.86 45.72))
-    (stroke (width 0) (type default))
-  )
   (wire (pts (xy 170.18 116.205) (xy 180.34 116.205))
     (stroke (width 0) (type default))
@@
     (effects (font (size 1.27 1.27)) (justify left bottom))
   )
-  (label "DI" (at 22.86 45.72 180) (fields_autoplaced)
-    (effects (font (size 1.27 1.27)) (justify right bottom))
-  )
   (label "SDA" (at 46.355 105.41 0) (fields_autoplaced)
     (effects (font (size 1.27 1.27)) (justify left bottom))
@@
   )
   (symbol (lib_id "Connector:Conn_01x03_Pin") (at 241.3 93.98 0) (mirror x) (unit 1)
-    (in_bom yes) (on_board yes) (dnp no)
+    (in_bom no) (on_board yes) (dnp no)
     (property "Reference" "J15" (at 241.935 100.965 0)
-      (effects (font (size 1.27 1.27)))
+      (effects (font (size 1.27 1.27)) hide)
     )
     (property "Value" "Conn_01x03_Pin" (at 240.03 88.265 0)
@@
   )
   (symbol (lib_id "Connector:Barrel_Jack") (at 23.495 165.735 0) (unit 1)
-    (in_bom yes) (on_board yes) (dnp no) (fields_autoplaced)
+    (in_bom no) (on_board yes) (dnp no) (fields_autoplaced)
     (property "Reference" "J13" (at 23.495 156.845 0)
-      (effects (font (size 1.27 1.27)))
+      (effects (font (size 1.27 1.27)) hide)
     )
     (property "Value" "Barrel_Jack" (at 23.495 159.385 0)
@@
   )
   (symbol (lib_id "Jumper:Jumper_2_Bridged") (at 104.14 170.18 0) (unit 1)
-    (in_bom yes) (on_board yes) (dnp no) (fields_autoplaced)
+    (in_bom no) (on_board yes) (dnp no) (fields_autoplaced)
     (property "Reference" "JP3" (at 104.14 165.1 0)
       (effects (font (size 1.27 1.27)))
@@
     (in_bom no) (on_board yes) (dnp no) (fields_autoplaced)
     (property "Reference" "JP1" (at 24.13 123.825 0)
-      (effects (font (size 1.27 1.27)))
+      (effects (font (size 1.27 1.27)) hide)
     )
     (property "Value" "Jumper_2_Open" (at 24.13 126.365 0)
@@
   )
   (symbol (lib_id "Connector:Conn_01x03_Pin") (at 264.16 93.98 0) (mirror x) (unit 1)
-    (in_bom yes) (on_board yes) (dnp no)
+    (in_bom no) (on_board yes) (dnp no)
     (property "Reference" "J17" (at 264.795 100.965 0)
-      (effects (font (size 1.27 1.27)))
+      (effects (font (size 1.27 1.27)) hide)
     )
     (property "Value" "Conn_01x03_Pin" (at 265.43 98.425 0)
@@
   )
   (symbol (lib_id "Device:C") (at 258.445 101.6 0) (unit 1)
-    (in_bom yes) (on_board yes) (dnp no)
+    (in_bom no) (on_board yes) (dnp no)
     (property "Reference" "C3" (at 261.62 100.33 0)
       (effects (font (size 1.27 1.27)) (justify left))
@@
   )
   (symbol (lib_id "Transistor_BJT:2N3904") (at 177.8 137.16 0) (unit 1)
-    (in_bom yes) (on_board yes) (dnp no) (fields_autoplaced)
+    (in_bom no) (on_board yes) (dnp no) (fields_autoplaced)
     (property "Reference" "Q2" (at 183.515 135.89 0)
-      (effects (font (size 1.27 1.27)) (justify left))
+      (effects (font (size 1.27 1.27)) (justify left) hide)
     )
     (property "Value" "2N3904" (at 183.515 138.43 0)
@@
       (effects (font (size 1.27 1.27)) (justify left) hide)
     )
+    (property "Customfield" "" (at 177.8 137.16 0)
+      (effects (font (size 1.27 1.27)) hide)
+    )
     (pin "3")
     (pin "1")
@@
   )
   (symbol (lib_id "Device:C") (at 278.765 100.33 0) (unit 1)
-    (in_bom yes) (on_board yes) (dnp no)
+    (in_bom no) (on_board yes) (dnp no)
     (property "Reference" "C4" (at 281.94 99.06 0)
       (effects (font (size 1.27 1.27)) (justify left))
